Commit message: Change model path

File: leo_erc_description/urdf/probe.urdf.xacro (robot description, xacro)
@@ -13,12 +13,18 @@
     <visual>
       <geometry>
-        <mesh filename="package://leo_erc_description/models/Probe.dae"/>
+        <mesh filename="package://leo_erc_description/models/Probe_v2.dae"/>
       </geometry>
     </visual>
     <collision>
       <geometry>
-        <mesh filename="package://leo_erc_description/models/Probe.dae"/>
+        <mesh filename="package://leo_erc_description/models/Probe_v2.dae"/>
       </geometry>
     </collision>
   </link>
+  <gazebo reference="probe_center">
+    <mu1>3.0</mu1>
+    <mu2>3.0</mu2>
+    <fdir1>0 1 0</fdir1>
+    <minDepth>0.002</minDepth>
+  </gazebo>
 </robot>

Commit message: Update probe properties

File: leo_erc_description/urdf/probe.urdf.xacro (robot description, xacro)
@@ -1,30 +1,32 @@
 <?xml version="1.0"?>
-<robot xmlns:xacro="http://ros.org/wiki/xacro"
-       name="probe_sim">
-  <link name="probe_center">
-    <inertial>
-      <mass value="0.01262"/>
-      <origin xyz="0 0 0"/>
-      <inertia
-        ixx="3.123e-6" ixy="0.0" ixz="0.0"
-        iyy="1.664e-6" iyz="0.0"
-        izz="1.664e-6"/>
-    </inertial>
-    <visual>
-      <geometry>
-        <mesh filename="package://leo_erc_description/models/Probe_v2.dae"/>
-      </geometry>
-    </visual>
-    <collision>
-      <geometry>
-        <mesh filename="package://leo_erc_description/models/Probe_v2.dae"/>
-      </geometry>
-    </collision>
-  </link>
-  <gazebo reference="probe_center">
-    <mu1>3.0</mu1>
-    <mu2>3.0</mu2>
-    <fdir1>0 1 0</fdir1>
-    <minDepth>0.002</minDepth>
-  </gazebo>
+<robot xmlns:xacro="http://ros.org/wiki/xacro" name="probe_sim">
+  <xacro:macro name="probe">
+    <link name="probe_center">
+      <inertial>
+        <mass value="0.00954"/>
+        <origin xyz="0 0 0"/>
+        <inertia
+          ixx="1.965e-6" ixy="0.0" ixz="0.0"
+          iyy="1.048e-6" iyz="0.0"
+          izz="1.048e-6"/>
+      </inertial>
+      <visual>
+        <geometry>
+          <mesh filename="package://leo_erc_description/models/Probe.dae"/>
+        </geometry>
+      </visual>
+      <collision>
+        <geometry>
+          <mesh filename="package://leo_erc_description/models/Probe.dae"/>
+        </geometry>
+      </collision>
+    </link>
+    <gazebo reference="probe_center">
+      <mu1>3.0</mu1>
+      <mu2>3.0</mu2>
+      <fdir1>0 1 0</fdir1>
+      <minDepth>0.002</minDepth>
+    </gazebo>
+  </xacro:macro>
+  <xacro:probe/>
 </robot>
