Commit message: Include URDF changes from upstream package

File: leo_erc_description/urdf/leo_macros.xacro (robot description, xacro)
@@ -6,5 +6,6 @@
                        footprint_link:=true
                        link_prefix:=''
-                       joint_prefix:=''">
+                       joint_prefix:=''
+                       imu_translation:='0.0628 -0.0314 -0.0393'">
     <xacro:macro name="rocker_link" params="name">
       <link name="${link_prefix}rocker_${name}_link">
@@ -118,4 +119,5 @@
     <link name="${link_prefix}camera_frame"/>
     <link name="${link_prefix}camera_optical_frame"/>
+    <link name="${link_prefix}imu_frame"/>
     <!-- JOINTS -->
     <xacro:if value="${footprint_link}">
@@ -197,4 +199,9 @@
       <parent link="${link_prefix}camera_frame"/>
       <child link="${link_prefix}camera_optical_frame"/>
+    </joint>
+    <joint name="${joint_prefix}imu_joint" type="fixed">
+      <origin xyz="${imu_translation}" rpy="0 0 0"/>
+      <parent link="${link_prefix}base_link"/>
+      <child link="${link_prefix}imu_frame"/>
     </joint>
   </xacro:macro>
@@ -322,4 +329,17 @@
       </plugin>
     </gazebo>
+    <gazebo reference="${link_prefix}imu_frame">
+      <sensor type="imu" name="leo_imu_sensor">
+        <update_rate>100</update_rate>
+        <plugin filename="libgazebo_ros_imu_sensor.so" name="imu_plugin">
+          <robotNamespace>${robot_ns}</robotNamespace>
+          <topicName>imu/data_raw</topicName>
+          <frameName>${link_prefix}imu_frame</frameName>
+          <updateRateHZ>100.0</updateRateHZ>
+          <gaussianNoise>0.01</gaussianNoise>
+          <initialOrientationAsReference>false</initialOrientationAsReference>
+        </plugin>
+      </sensor>
+    </gazebo>
     <!-- ros_control plugin -->
     <gazebo>
